Commit message: Creating launch files and using remap

File: src/my_r2d2/urdf/r2d2.urdf.xacro (robot description, xacro)
@@ -37,4 +37,11 @@
     <xacro:default_inertial mass="10"/>
   </link>
+  <link name="base_footprint">
+  </link>
+  <joint name="footprint_to_base" type="fixed">
+      <parent link="base_footprint"/>
+      <child link="base_link"/>
+      <origin xyz="0 0 ${wheeldiam+bodylen/2+0.1}" />
+  </joint>
   <xacro:macro name="wheel" params="prefix suffix reflect">
     <link name="${prefix}_${suffix}_wheel">
