Commit message: Trying camera and tag tracking

File: src/my_r2d2/urdf/r2d2.urdf (robot description, URDF)
Before this commit: robot physics, 16 links, 15 joints
Links:
- added link eye
Joints:
- added joint eyebox: type fixed, parent box, child eye, origin rpy=0 1.57075 0

File: src/my_r2d2/urdf/r2d2.urdf.xacro (robot description, xacro)
@@ -220,3 +220,10 @@
     <origin xyz="${.707*width+0.04} 0 ${.707*width}"/>
   </joint>
+<link name="eye">
+  </link>
+<joint name="eyebox" type="fixed">
+    <parent link="box"/>
+    <child link="eye"/>
+ <origin rpy="-1.57075 0 -1.57075"/>
+  </joint>
 </robot>
